Commit message: Increase inertias to 1e-2 for numerical stability

File: urdf/humanoid.xacro (robot description, xacro)
@@ -13,6 +13,6 @@
   <link name="${parent}_${child}_link1">
     <inertial>
-      <mass value="1e-09" />
-      <inertia ixx="1e-09" ixy="0" ixz="0" iyy="1e-09" iyz="0" izz="1e-09" />
+      <mass value="1e-02" />
+      <inertia ixx="1e-02" ixy="0" ixz="0" iyy="1e-02" iyz="0" izz="1e-02" />
     </inertial>
   </link>
@@ -24,6 +24,6 @@
   <link name="${parent}_${child}_link2">
     <inertial>
-      <mass value="1e-09" />
-      <inertia ixx="1e-09" ixy="0" ixz="0" iyy="1e-09" iyz="0" izz="1e-09" />
+      <mass value="1e-02" />
+      <inertia ixx="1e-02" ixy="0" ixz="0" iyy="1e-02" iyz="0" izz="1e-02" />
     </inertial>
 	<visual>
@@ -41,6 +41,6 @@
   <link name="${parent}_${child}_link3">
     <inertial>
-      <mass value="1e-09" />
-      <inertia ixx="1e-09" ixy="0" ixz="0" iyy="1e-09" iyz="0" izz="1e-09" />
+      <mass value="1e-02" />
+      <inertia ixx="1e-02" ixy="0" ixz="0" iyy="1e-02" iyz="0" izz="1e-02" />
     </inertial>
   </link>

Commit message: Fix order of links and joints

File: urdf/humanoid.xacro (robot description, xacro)
@@ -5,10 +5,4 @@
 </material>
 <xacro:macro name="ball_joint" params="parent child *origin">
-  <joint name="${parent}_${child}_joint1" type="continuous">
-	<xacro:insert_block name="origin"/>
-    <parent link="${parent}"/>
-    <child link="${parent}_${child}_link1"/>
-    <axis xyz="1 0 0" />
-  </joint>
   <link name="${parent}_${child}_link1">
     <inertial>
@@ -17,8 +11,9 @@
     </inertial>
   </link>
-  <joint name="${parent}_${child}_joint2" type="continuous">
-    <parent link="${parent}_${child}_link1"/>
-    <child link="${parent}_${child}_link2"/>
-    <axis xyz="0 1 0" />
+  <joint name="${parent}_${child}_joint1" type="continuous">
+	<xacro:insert_block name="origin"/>
+    <parent link="${parent}"/>
+    <child link="${parent}_${child}_link1"/>
+    <axis xyz="1 0 0" />
   </joint>
   <link name="${parent}_${child}_link2">
@@ -34,4 +29,9 @@
 	</visual>
   </link>
+  <joint name="${parent}_${child}_joint2" type="continuous">
+    <parent link="${parent}_${child}_link1"/>
+    <child link="${parent}_${child}_link2"/>
+    <axis xyz="0 1 0" />
+  </joint>
   <joint name="${parent}_${child}_joint3" type="continuous">
     <parent link="${parent}_${child}_link2"/>
