Commit message: add motion data & work on xacro

File: urdf/humanoid.urdf (robot description, URDF)
Before this commit: robot dumpUrdf, 41 links, 40 joints
Links:
- added link chest_left_shoulder_link0, mass 5e-4
- added link chest_neck_link0, mass 5e-4
- added link chest_right_shoulder_link0, mass 5e-4
- added link left_knee_left_ankle_link0, mass 5e-4
- added link right_knee_right_ankle_link0, mass 5e-4
- added link root_chest_link0, mass 5e-4
- added link root_left_hip_link0, mass 5e-4
- added link root_right_hip_link0, mass 5e-4
- link chest: geometry collision sphere radius=0.11; visual sphere radius=0.11
- link chest_left_shoulder_link2: geometry visual sphere radius=0.05
- link chest_neck_link2: geometry visual sphere radius=0.05
- link chest_right_shoulder_link2: geometry visual sphere radius=0.05
- link left_ankle: geometry collision box size=0.177 0.055 0.09; visual box size=0.177 0.055 0.09
- link left_elbow: geometry collision cylinder length=0.135 radius=0.04; visual cylinder length=0.135 radius=0.04
- link left_hip: geometry collision cylinder length=0.3 radius=0.055; visual cylinder length=0.3 radius=0.055
- link left_knee: geometry collision cylinder length=0.31 radius=0.05; visual cylinder length=0.31 radius=0.05
- link left_knee_left_ankle_link2: geometry visual sphere radius=0.05
- link left_shoulder: geometry collision cylinder length=0.18 radius=0.045; visual cylinder length=0.18 radius=0.045
- link left_wrist: geometry collision sphere radius=0.04; visual sphere radius=0.04
- link neck: geometry collision sphere radius=0.1025; visual sphere radius=0.1025
- link right_ankle: geometry collision box size=0.177 0.055 0.09; visual box size=0.177 0.055 0.09
- link right_elbow: geometry collision cylinder length=0.135 radius=0.04; visual cylinder length=0.135 radius=0.04
- link right_hip: geometry collision cylinder length=0.3 radius=0.055; visual cylinder length=0.3 radius=0.055
- link right_knee: geometry collision cylinder length=0.31 radius=0.05; visual cylinder length=0.31 radius=0.05
- link right_knee_right_ankle_link2: geometry visual sphere radius=0.05
- link right_shoulder: geometry collision cylinder length=0.18 radius=0.045; visual cylinder length=0.18 radius=0.045
- link right_wrist: geometry collision sphere radius=0.04; visual sphere radius=0.04
- link root: geometry collision sphere radius=0.09; visual sphere radius=0.09
- link root_chest_link2: geometry visual sphere radius=0.05
- link root_left_hip_link2: geometry visual sphere radius=0.05
- link root_right_hip_link2: geometry visual sphere radius=0.05
Joints:
- added joint chest_left_shoulder_dummy1: type fixed, parent chest, child chest_left_shoulder_link0, origin xyz=-0.02405 0.24350 -0.18311 rpy=0 0 0
- added joint chest_neck_dummy1: type fixed, parent chest, child chest_neck_link0, origin xyz=0.000000 0.223894 0.000000 rpy=0 0 0
- added joint chest_right_shoulder_dummy1: type fixed, parent chest, child chest_right_shoulder_link0, origin xyz=-0.02406 0.24350 0.18311 rpy=0 0 0
- added joint left_knee_left_ankle_dummy1: type fixed, parent left_knee, child left_knee_left_ankle_link0, origin xyz=0.000000 -0.40987 0.000000 rpy=0 0 0
- added joint right_knee_right_ankle_dummy1: type fixed, parent right_knee, child right_knee_right_ankle_link0, origin xyz=0.000000 -0.409870 0.000000 rpy=0 0 0
- added joint root_chest_dummy1: type fixed, parent root, child root_chest_link0, origin xyz=0.000000 0.236151 0.000000 rpy=0 0 0
- added joint root_left_hip_dummy1: type fixed, parent root, child root_left_hip_link0, origin xyz=0.000000 0.000000 -0.084887 rpy=0 0 0
- added joint root_right_hip_dummy1: type fixed, parent root, child root_right_hip_link0, origin xyz=0.000000 0.000000 0.084887 rpy=0 0 0
- joint chest_left_shoulder_joint1: origin xyz=-0.096200 0.974000 -0.732440 rpy=0 0 0 -> (none); parent chest -> chest_left_shoulder_link0
- joint chest_neck_joint1: origin xyz=0.000000 0.895576 0.000000 rpy=0 0 0 -> (none); parent chest -> chest_neck_link0
- joint chest_right_shoulder_joint1: origin xyz=-0.096200 0.974000 0.732440 rpy=0 0 0 -> (none); parent chest -> chest_right_shoulder_link0
- joint left_elbow: origin xyz=0.000000 -1.099152 0.000000 rpy=0 0 0 -> xyz=0.000000 -0.274788 0.000000 rpy=0 0 0
- joint left_knee: origin xyz=0.000000 -1.686184 0.000000 rpy=0 0 0 -> xyz=0.000000 -0.421546 0.000000 rpy=0 0 0
- joint left_knee_left_ankle_joint1: origin xyz=0.000000 -1.639480 0.000000 rpy=0 0 0 -> (none); parent left_knee -> left_knee_left_ankle_link0
- joint left_wrist_joint: origin xyz=0.000000 -1.035788 0.000000 rpy=0 0 0 -> xyz=0.000000 -0.258947 0.000000 rpy=0 0 0
- joint right_elbow: origin xyz=0.000000 -1.099152 0.000000 rpy=0 0 0 -> xyz=0.000000 -0.274788 0.000000 rpy=0 0 0
- joint right_knee: origin xyz=0.000000 -1.686184 0.000000 rpy=0 0 0 -> xyz=0.000000 -0.421546 0.000000 rpy=0 0 0
- joint right_knee_right_ankle_joint1: origin xyz=0.000000 -1.639480 0.000000 rpy=0 0 0 -> (none); parent right_knee -> right_knee_right_ankle_link0
- joint right_wrist: origin xyz=0.000000 -1.035788 0.000000 rpy=0 0 0 -> xyz=0.000000 -0.258947 0.000000 rpy=0 0 0
- joint root_chest_joint1: origin xyz=0.000000 0.944604 0.000000 rpy=0 0 0 -> (none); parent root -> root_chest_link0
- joint root_left_hip_joint1: origin xyz=0.000000 0.000000 -0.339548 rpy=0 0 0 -> (none); parent root -> root_left_hip_link0
- joint root_right_hip_joint1: origin xyz=0.000000 0.000000 0.339548 rpy=0 0 0 -> (none); parent root -> root_right_hip_link0

File: urdf/humanoid.xacro (robot description, xacro)
@@ -1,4 +1,7 @@
 <?xml version="1.0"?>
 <robot  xmlns:xacro="http://www.ros.org/wiki/xacro"  name="dumpUrdf">
+<material name="orange">
+  <color rgba="${255/255} ${108/255} ${10/255} 1.0"/>
+</material>
 <xacro:macro name="ball_joint" params="parent child *origin">
   <joint name="${parent}_${child}_joint1" type="continuous">
@@ -24,4 +27,10 @@
       <inertia ixx="5e-4" ixy="0" ixz="0" iyy="5e-5" iyz="0" izz="5e-4" />
     </inertial>
+	<visual>
+		<geometry>
+			<sphere radius="0.05"  />
+		</geometry>
+		<material name="orange"/>
+	</visual>
   </link>
   <joint name="${parent}_${child}_joint3" type="continuous">
@@ -45,10 +54,10 @@
 		<xacro:insert_block name="origin"/>
 		<geometry>
-			<sphere radius = "${radius}"/>
+			<sphere radius = "${radius/2}"/>
 		</geometry>
 	</collision>
 	<visual>
 		<geometry>
-			<sphere radius="${radius}"/>
+			<sphere radius="${radius/2}"/>
 		</geometry>
 	</visual>
@@ -58,5 +67,5 @@
 		<xacro:insert_block name="origin"/>
 		<geometry>
-			<cylinder length="${length}" radius = "${radius}"/>
+			<cylinder length="${length}" radius = "${radius/2}"/>
 		</geometry>
 	</collision>
@@ -64,5 +73,5 @@
 		<xacro:insert_block name="origin"/>
 		<geometry>
-			<cylinder length="${length}" radius="${radius}"/>
+			<cylinder length="${length}" radius="${radius/2}"/>
 		</geometry>
 	</visual>
@@ -93,17 +102,11 @@
 	<link name="root" >
 		<inertial>
-			<origin rpy = "0 0 0" xyz = "0.000000 0.280000 0.000000" />
+			<origin rpy = "0 0 0" xyz = "0.0 0.07 0.0" />
 			<mass value = "6.000000" />
 			<inertia ixx = "0.1" ixy = "0" ixz = "0" iyy = "0.1" iyz = "0" izz = "0.1" />
 		</inertial>
-		<xacro:sphere_v_c radius="0.36">
-			<origin rpy = "0 0 0" xyz = "0.000000 0.280000 0.000000" />
-		</xacro:sphere_v_c>
-		<!--<collision>
-				<origin rpy = "0 0 0" xyz = "0.000000 0.280000 0.000000" />
-			<geometry>
-				<sphere radius = "0.360000" />
-			</geometry>
-		</collision>-->
+		<xacro:sphere_v_c radius="0.18">
+			<origin rpy = "0 0 0" xyz = "0.000000 0.070000 0.000000" />
+		</xacro:sphere_v_c>
 	</link>
 	<joint name="root" type="fixed" >
@@ -114,157 +117,93 @@
 	<link name="chest" >
 		<inertial>
-				<origin rpy = "0 0 0" xyz = "0.000000 0.480000 0.000000" />
-			 <mass value = "14.000000" />
-			<inertia ixx = "0.1" ixy = "0" ixz = "0" iyy = "0.1" iyz = "0" izz = "0.1" />
-		</inertial>
-		<xacro:sphere_v_c radius="0.44">
-			<origin rpy = "0 0 0" xyz = "0.000000 0.480000 0.000000" />
-		</xacro:sphere_v_c>
-		<!--<collision>
-				<origin rpy = "0 0 0" xyz = "0.000000 0.480000 0.000000" />
-			<geometry>
-				<sphere radius = "0.440000" />
-			</geometry>
-		</collision>-->
-	</link>
-    <!-- Spherical joints start -->
+			<origin rpy = "0 0 0" xyz = "0.000000 0.120000 0.000000" />
+			<mass value = "14.000000" />
+			<inertia ixx = "0.1" ixy = "0" ixz = "0" iyy = "0.1" iyz = "0" izz = "0.1" />
+		</inertial>
+		<xacro:sphere_v_c radius="0.22">
+			<origin rpy = "0 0 0" xyz = "0.000000 0.120000 0.000000" />
+		</xacro:sphere_v_c>
+	</link>
 	<xacro:ball_joint parent="root" child="chest">
-		<origin rpy = "0 0 0" xyz = "0.000000 0.944604 0.000000" />
-	</xacro:ball_joint>
-    <!-- Spherical joints end -->
+		<origin rpy = "0 0 0" xyz = "0.000000 0.236151 0.000000" />
+	</xacro:ball_joint>
 	<link name="neck" >
 		<inertial>
-				<origin rpy = "0 0 0" xyz = "0.000000 0.700000 0.000000" />
-			 <mass value = "2.000000" />
-			<inertia ixx = "0.1" ixy = "0" ixz = "0" iyy = "0.1" iyz = "0" izz = "0.1" />
-		</inertial>
-		<xacro:sphere_v_c radius="0.41">
-			<origin rpy = "0 0 0" xyz = "0.000000 0.70000 0.000000" />
-		</xacro:sphere_v_c>
-		<!--<collision>
-				<origin rpy = "0 0 0" xyz = "0.000000 0.700000 0.000000" />
-			<geometry>
-				<sphere radius = "0.410000" />
-			</geometry>
-		</collision>-->
+			<origin rpy = "0 0 0" xyz = "0.0 0.175 0.0" />
+			<mass value = "2.000000" />
+			<inertia ixx = "0.1" ixy = "0" ixz = "0" iyy = "0.1" iyz = "0" izz = "0.1" />
+		</inertial>
+		<xacro:sphere_v_c radius="0.205">
+			<origin rpy = "0 0 0" xyz = "0.0 0.175 0.0" />
+		</xacro:sphere_v_c>
 	</link>
 	<xacro:ball_joint parent="chest" child="neck" >
-		<origin rpy = "0 0 0" xyz = "0.000000 0.895576 0.000000" />
-	</xacro:ball_joint>
-	<!--<joint name="neck" type="spherical" >
-		<parent link="chest" />
-		<child link="neck" />
-				<origin rpy = "0 0 0" xyz = "0.000000 0.895576 0.000000" />
-	</joint>-->
+		<origin rpy = "0 0 0" xyz = "0.000000 0.223894 0.000000" />
+	</xacro:ball_joint>
 	<link name="right_hip" >
 		<inertial>
-				<origin rpy = "0 0 0" xyz = "0.000000 -0.840000 0.000000" />
-			 <mass value = "4.500000" />
-			<inertia ixx = "0.1" ixy = "0" ixz = "0" iyy = "0.1" iyz = "0" izz = "0.1" />
-		</inertial>
-		<xacro:cylinder_v_c radius="0.22" length="1.2">
-				<origin rpy = "-1.570796 0 0" xyz = "0.000000 -0.840000 0.000000" />
-		</xacro:cylinder_v_c>
-		<!--<collision>
-				<origin rpy = "-1.570796 0 0" xyz = "0.000000 -0.840000 0.000000" />
-			<geometry>
-				<cylinder length="1.200000" radius="0.220000"/>
-			</geometry>
-		</collision>-->
+			<origin rpy = "0 0 0" xyz = "0.000000 -0.210000 0.000000" />
+			<mass value = "4.500000" />
+			<inertia ixx = "0.1" ixy = "0" ixz = "0" iyy = "0.1" iyz = "0" izz = "0.1" />
+		</inertial>
+		<xacro:cylinder_v_c radius="0.11" length="0.3">
+				<origin rpy = "${pi/2} 0 0" xyz = "0.000000 -0.210000 0.000000" />
+		</xacro:cylinder_v_c>
 	</link>
 	<xacro:ball_joint parent="root" child="right_hip">
-		<origin rpy = "0 0 0" xyz = "0.000000 0.000000 0.339548" />
-	</xacro:ball_joint>
-	<!--<joint name="right_hip" type="spherical" >
-		<parent link="root" />
-		<child link="right_hip" />
-				<origin rpy = "0 0 0" xyz = "0.000000 0.000000 0.339548" />
-	</joint>-->
+		<origin rpy = "0 0 0" xyz = "0.000000 0.000000 0.084887" />
+	</xacro:ball_joint>
 	<link name="right_knee" >
 		<inertial>
-				<origin rpy = "0 0 0" xyz = "0.000000 -0.800000 0.000000" />
-			 <mass value = "3.000000" />
-			<inertia ixx = "0.1" ixy = "0" ixz = "0" iyy = "0.1" iyz = "0" izz = "0.1" />
-		</inertial>
-		<xacro:cylinder_v_c length="1.240000" radius="0.200000">
-				<origin rpy = "-1.570796 0 0" xyz = "0.000000 -0.800000 0.000000" />
-		</xacro:cylinder_v_c>
-		<!--<collision>
-				<origin rpy = "-1.570796 0 0" xyz = "0.000000 -0.800000 0.000000" />
-			<geometry>
-				<cylinder length="1.240000" radius="0.200000"/>
-			</geometry>
-		</collision>-->
+			<origin rpy = "0 0 0" xyz = "0.000000 -0.200000 0.000000" />
+			<mass value = "3.000000" />
+			<inertia ixx = "0.1" ixy = "0" ixz = "0" iyy = "0.1" iyz = "0" izz = "0.1" />
+		</inertial>
+		<xacro:cylinder_v_c length="0.31" radius="0.1">
+			<origin rpy = "${pi/2} 0 0" xyz = "0.000000 -0.200000 0.000000" />
+		</xacro:cylinder_v_c>
 	</link>
 	<joint name="right_knee" type="revolute" >
 		<parent link="right_hip" />
 		<child link="right_knee" />
-		 <limit effort="1000.0" lower="-3.14" upper="0." velocity="0.5"/>
-			<origin rpy = "0 0 0" xyz = "0.000000 -1.686184 0.000000" />
+		<limit effort="1000.0" lower="-3.14" upper="0." velocity="0.5"/>
+		<origin rpy = "0 0 0" xyz = "0.000000 -0.421546 0.000000" />
 		<axis xyz = "0.000000 0.000000 1.000000" />
 	</joint>
 	<link name="right_ankle" >
 		<inertial>
-				<origin rpy = "0 0 0" xyz = "0.180000 -0.090000 0.000000" />
-			 <mass value = "1.000000" />
-			<inertia ixx = "0.1" ixy = "0" ixz = "0" iyy = "0.1" iyz = "0" izz = "0.1" />
-		</inertial>
-		<xacro:box_v_c x="0.708" y="0.22" z = "0.36">
-				<origin rpy = "0 0 0" xyz = "0.180000 -0.090000 0.000000" />
+			<origin rpy = "0 0 0" xyz = "0.045 -0.00225 0.000000" />
+			<mass value = "1.000000" />
+			<inertia ixx = "0.1" ixy = "0" ixz = "0" iyy = "0.1" iyz = "0" izz = "0.1" />
+		</inertial>
+		<xacro:box_v_c x="0.177" y="0.055" z = "0.09">
+				<origin rpy = "0 0 0" xyz = "0.045 -0.00225 0.000000"  />
 		</xacro:box_v_c>
-		<!--<collision>
-				<origin rpy = "0 0 0" xyz = "0.180000 -0.090000 0.000000" />
-			<geometry>
-				<box size="0.708000 0.220000 0.360000" />
-			</geometry>
-		</collision>-->
 	</link>
 	<xacro:ball_joint parent="right_knee" child="right_ankle">
-		<origin rpy = "0 0 0" xyz = "0.000000 -1.639480 0.000000" />
-	</xacro:ball_joint>
-	<!--<joint name="right_ankle" type="spherical" >
-		<parent link="right_knee" />
-		<child link="right_ankle" />
-				<origin rpy = "0 0 0" xyz = "0.000000 -1.639480 0.000000" />
-	</joint>-->
+		<origin rpy = "0 0 0" xyz = "0.000000 -0.409870 0.000000" />
+	</xacro:ball_joint>
 	<link name="right_shoulder" >
 		<inertial>
-				<origin rpy = "0 0 0" xyz = "0.000000 -0.560000 0.000000" />
-			 <mass value = "1.500000" />
-			<inertia ixx = "0.1" ixy = "0" ixz = "0" iyy = "0.1" iyz = "0" izz = "0.1" />
-		</inertial>
-		<xacro:cylinder_v_c length="0.720000" radius="0.180000">
-				<origin rpy = "-1.570796 0 0" xyz = "0.000000 -0.560000 0.000000" />
-		</xacro:cylinder_v_c>
-		<!--<collision>
-				<origin rpy = "-1.570796 0 0" xyz = "0.000000 -0.560000 0.000000" />
-			<geometry>
-				<cylinder length="0.720000" radius="0.180000"/>
-			</geometry>
-		</collision>-->
+			<origin rpy = "0 0 0" xyz = "0.000000 -0.140000 0.000000" />
+			<mass value = "1.500000" />
+			<inertia ixx = "0.1" ixy = "0" ixz = "0" iyy = "0.1" iyz = "0" izz = "0.1" />
+		</inertial>
+		<xacro:cylinder_v_c length="0.18" radius="0.09">
+			<origin rpy = "${pi/2} 0 0" xyz = "0.000000 -0.140000 0.000000" />
+		</xacro:cylinder_v_c>
 	</link>
 	<xacro:ball_joint parent="chest" child="right_shoulder">
-		<origin rpy = "0 0 0" xyz = "-0.096200 0.974000 0.732440" />
-	</xacro:ball_joint>
-	<!--<joint name="right_shoulder" type="spherical" >
-		<parent link="chest" />
-		<child link="right_shoulder" />
-				<origin rpy = "0 0 0" xyz = "-0.096200 0.974000 0.732440" />
-	</joint>-->
+		<origin rpy = "0 0 0" xyz = "-0.02406 0.24350 0.18311" />
+	</xacro:ball_joint>
 	<link name="right_elbow" >
 		<inertial>
-				<origin rpy = "0 0 0" xyz = "0.000000 -0.480000 0.000000" />
-			 <mass value = "1.000000" />
-			<inertia ixx = "0.1" ixy = "0" ixz = "0" iyy = "0.1" iyz = "0" izz = "0.1" />
-		</inertial>
-		<xacro:cylinder_v_c length="0.540000" radius="0.160000">
-				<origin rpy = "-1.570796 0 0" xyz = "0.000000 -0.480000 0.000000" />
-		</xacro:cylinder_v_c>
-		<!--<collision>
-				<origin rpy = "-1.570796 0 0" xyz = "0.000000 -0.480000 0.000000" />
-			<geometry>
-				<cylinder length="0.540000" radius="0.160000"/>
-			</geometry>
-		</collision>-->
+			<origin rpy = "0 0 0" xyz = "0.000000 -0.120000 0.000000" />
+			<mass value = "1.000000" />
+			<inertia ixx = "0.1" ixy = "0" ixz = "0" iyy = "0.1" iyz = "0" izz = "0.1" />
+		</inertial>
+		<xacro:cylinder_v_c length="0.135" radius="0.08">
+				<origin rpy = "${pi/2} 0 0" xyz = "0.0 -0.12 0.0" />
+		</xacro:cylinder_v_c>
 	</link>
 	<joint name="right_elbow" type="revolute" >
@@ -272,67 +211,44 @@
 		<child link="right_elbow" />
 		<limit effort="1000.0" lower="0" upper="3.14" velocity="0.5"/>
-				<origin rpy = "0 0 0" xyz = "0.000000 -1.099152 0.000000" />
+		<origin rpy = "0 0 0" xyz = "0.000000 -0.274788 0.000000" />
 		<axis xyz = "0.000000 0.000000 1.000000" />
 	</joint>
 	<link name="right_wrist" >
 		<inertial>
-				<origin rpy = "0 0 0" xyz = "0.000000 0.000000 0.000000" />
-			 <mass value = "0.500000" />
-			<inertia ixx = "0.1" ixy = "0" ixz = "0" iyy = "0.1" iyz = "0" izz = "0.1" />
-		</inertial>
-		<xacro:sphere_v_c radius="0.16">
-				<origin rpy = "0 0 0" xyz = "0.000000 0.000000 0.000000" />
-		</xacro:sphere_v_c>
-		<!--<collision>
-				<origin rpy = "0 0 0" xyz = "0.000000 0.000000 0.000000" />
-			<geometry>
-				<sphere radius = "0.160000" />
-			</geometry>
-		</collision>-->
+			<origin rpy = "0 0 0" xyz = "0.000000 0.000000 0.000000" />
+			<mass value = "0.500000" />
+			<inertia ixx = "0.1" ixy = "0" ixz = "0" iyy = "0.1" iyz = "0" izz = "0.1" />
+		</inertial>
+		<xacro:sphere_v_c radius="0.08">
+			<origin rpy = "0 0 0" xyz = "0.000000 0.000000 0.000000" />
+		</xacro:sphere_v_c>
 	</link>
 	<joint name="right_wrist" type="fixed" >
 		<parent link="right_elbow" />
 		<child link="right_wrist" />
-				<origin rpy = "0 0 0" xyz = "0.000000 -1.035788 0.000000" />
+		<origin rpy = "0 0 0" xyz = "0.000000 -0.258947 0.000000" />
 	</joint>
 	<link name="left_hip" >
 		<inertial>
-				<origin rpy = "0 0 0" xyz = "0.000000 -0.840000 0.000000" />
-			 <mass value = "4.500000" />
-			<inertia ixx = "0.1" ixy = "0" ixz = "0" iyy = "0.1" iyz = "0" izz = "0.1" />
-		</inertial>
-		<xacro:cylinder_v_c length="1.200000" radius="0.220000">
-				<origin rpy = "-1.570796 0 0" xyz = "0.000000 -0.840000 0.000000" />
-		</xacro:cylinder_v_c>
-		<!--<collision>
-				<origin rpy = "-1.570796 0 0" xyz = "0.000000 -0.840000 0.000000" />
-			<geometry>
-				<cylinder length="1.200000" radius="0.220000"/>
-			</geometry>
-		</collision>-->
+			<origin rpy = "0 0 0" xyz = "0.000000 -0.210000 0.000000" />
+			<mass value = "4.500000" />
+			<inertia ixx = "0.1" ixy = "0" ixz = "0" iyy = "0.1" iyz = "0" izz = "0.1" />
+		</inertial>
+		<xacro:cylinder_v_c length="0.3" radius="0.11">
+				<origin rpy = "${pi/2} 0 0" xyz = "0.000000 -0.210000 0.000000" />
+		</xacro:cylinder_v_c>
 	</link>
 	<xacro:ball_joint parent="root" child="left_hip">
-		<origin rpy = "0 0 0" xyz = "0.000000 0.000000 -0.339548" />
-	</xacro:ball_joint>
-	<!--<joint name="left_hip" type="spherical" >
-		<parent link="root" />
-		<child link="left_hip" />
-				<origin rpy = "0 0 0" xyz = "0.000000 0.000000 -0.339548" />
-	</joint>-->
+		<origin rpy = "0 0 0" xyz = "0.000000 0.000000 -0.084887" />
+	</xacro:ball_joint>
 	<link name="left_knee" >
 		<inertial>
-				<origin rpy = "0 0 0" xyz = "0.000000 -0.800000 0.000000" />
+				<origin rpy = "0 0 0" xyz = "0.000000 -0.200000 0.000000" />
 			 <mass value = "3.000000" />
 			<inertia ixx = "0.1" ixy = "0" ixz = "0" iyy = "0.1" iyz = "0" izz = "0.1" />
 		</inertial>
-		<xacro:cylinder_v_c length="1.240000" radius="0.20000">
-				<origin rpy = "-1.570796 0 0" xyz = "0.000000 -0.800000 0.000000" />
-		</xacro:cylinder_v_c>
-		<!--<collision>
-				<origin rpy = "-1.570796 0 0" xyz = "0.000000 -0.800000 0.000000" />
-			<geometry>
-				<cylinder length="1.240000" radius="0.200000"/>
-			</geometry>
-		</collision>-->
+		<xacro:cylinder_v_c length="0.31" radius="0.10000">
+				<origin rpy = "${pi/2} 0 0" xyz = "0.000000 -0.200000 0.000000" />
+		</xacro:cylinder_v_c>
 	</link>
 	<joint name="left_knee" type="revolute" >
@@ -340,70 +256,42 @@
 		<child link="left_knee" />
 		<limit effort="1000.0" lower="-3.14" upper="0." velocity="0.5"/>
-				<origin rpy = "0 0 0" xyz = "0.000000 -1.686184 0.000000" />
+		<origin rpy = "0 0 0" xyz = "0.000000 -0.421546 0.000000" />
 		<axis xyz = "0.000000 0.000000 1.000000" />
 	</joint>
 	<link name="left_ankle" >
 		<inertial>
-				<origin rpy = "0 0 0" xyz = "0.180000 -0.090000 0.000000" />
-			 <mass value = "1.000000" />
-			<inertia ixx = "0.1" ixy = "0" ixz = "0" iyy = "0.1" iyz = "0" izz = "0.1" />
-		</inertial>
-		<xacro:box_v_c x="0.708" y="0.22" z = "0.36">
-				<origin rpy = "0 0 0" xyz = "0.180000 -0.090000 0.000000" />
+			<origin rpy = "0 0 0" xyz = "0.045 -0.00225 0.0" />
+			<mass value = "1.000000" />
+			<inertia ixx = "0.1" ixy = "0" ixz = "0" iyy = "0.1" iyz = "0" izz = "0.1" />
+		</inertial>
+		<xacro:box_v_c x="0.177" y="0.055" z = "0.09">
+				<origin rpy = "0 0 0" xyz = "0.045 -0.00225 0.0" />
 		</xacro:box_v_c>
-		<!--<collision>
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