Commit message: change urdf model

File: urdf/humanoid.urdf (robot description, URDF)
Before this commit: robot dumpUrdf, 49 links, 48 joints
Links:
- removed link chest_left_shoulder_link0
- removed link chest_neck_link0
- removed link chest_right_shoulder_link0
- removed link left_knee_left_ankle_link0
- removed link right_knee_right_ankle_link0
- removed link root_chest_link0
- removed link root_left_hip_link0
- removed link root_right_hip_link0
- link chest_left_shoulder_link1: mass 5e-4 -> 1e-09
- link chest_left_shoulder_link2: mass 5e-4 -> 1e-09
- link chest_left_shoulder_link3: mass 5e-4 -> 1e-09
- link chest_neck_link1: mass 5e-4 -> 1e-09
- link chest_neck_link2: mass 5e-4 -> 1e-09
- link chest_neck_link3: mass 5e-4 -> 1e-09
- link chest_right_shoulder_link1: mass 5e-4 -> 1e-09
- link chest_right_shoulder_link2: mass 5e-4 -> 1e-09
- link chest_right_shoulder_link3: mass 5e-4 -> 1e-09
- link left_elbow: geometry collision cylinder length=0.10125 radius=0.02; visual cylinder length=0.135 radius=0.04
- link left_hip: geometry collision cylinder length=0.225 radius=0.0275; visual cylinder length=0.3 radius=0.055
- link left_knee: geometry collision cylinder length=0.2325 radius=0.025; visual cylinder length=0.31 radius=0.05
- link left_knee_left_ankle_link1: mass 5e-4 -> 1e-09
- link left_knee_left_ankle_link2: mass 5e-4 -> 1e-09
- link left_knee_left_ankle_link3: mass 5e-4 -> 1e-09
- link left_shoulder: geometry collision cylinder length=0.135 radius=0.0225; visual cylinder length=0.18 radius=0.045
- link right_elbow: geometry collision cylinder length=0.10125 radius=0.02; visual cylinder length=0.135 radius=0.04
- link right_hip: geometry collision cylinder length=0.225 radius=0.0275; visual cylinder length=0.3 radius=0.055
- link right_knee: geometry collision cylinder length=0.2325 radius=0.025; visual cylinder length=0.31 radius=0.05
- link right_knee_right_ankle_link1: mass 5e-4 -> 1e-09
- link right_knee_right_ankle_link2: mass 5e-4 -> 1e-09
- link right_knee_right_ankle_link3: mass 5e-4 -> 1e-09
- link right_shoulder: geometry collision cylinder length=0.135 radius=0.0225; visual cylinder length=0.18 radius=0.045
- link root_chest_link1: mass 5e-4 -> 1e-09
- link root_chest_link2: mass 5e-4 -> 1e-09
- link root_chest_link3: mass 5e-4 -> 1e-09
- link root_left_hip_link1: mass 5e-4 -> 1e-09
- link root_left_hip_link2: mass 5e-4 -> 1e-09
- link root_left_hip_link3: mass 5e-4 -> 1e-09
- link root_right_hip_link1: mass 5e-4 -> 1e-09
- link root_right_hip_link2: mass 5e-4 -> 1e-09
- link root_right_hip_link3: mass 5e-4 -> 1e-09
Joints:
- removed joint chest_left_shoulder_dummy1
- removed joint chest_neck_dummy1
- removed joint chest_right_shoulder_dummy1
- removed joint left_knee_left_ankle_dummy1
- removed joint right_knee_right_ankle_dummy1
- removed joint root_chest_dummy1
- removed joint root_left_hip_dummy1
- removed joint root_right_hip_dummy1
- joint chest_left_shoulder_joint1: origin (none) -> xyz=-0.02405 0.24350 -0.18311 rpy=0 0 0; parent chest_left_shoulder_link0 -> chest
- joint chest_neck_joint1: origin (none) -> xyz=0.000000 0.223894 0.000000 rpy=0 0 0; parent chest_neck_link0 -> chest
- joint chest_right_shoulder_joint1: origin (none) -> xyz=-0.02406 0.24350 0.18311 rpy=0 0 0; parent chest_right_shoulder_link0 -> chest
- joint left_knee_left_ankle_joint1: origin (none) -> xyz=0.000000 -0.40987 0.000000 rpy=0 0 0; parent left_knee_left_ankle_link0 -> left_knee
- joint right_knee_right_ankle_joint1: origin (none) -> xyz=0.000000 -0.409870 0.000000 rpy=0 0 0; parent right_knee_right_ankle_link0 -> right_knee
- joint root_chest_joint1: origin (none) -> xyz=0.000000 0.236151 0.000000 rpy=0 0 0; parent root_chest_link0 -> root
- joint root_left_hip_joint1: origin (none) -> xyz=0.000000 0.000000 -0.084887 rpy=0 0 0; parent root_left_hip_link0 -> root
- joint root_right_hip_joint1: origin (none) -> xyz=0.000000 0.000000 0.084887 rpy=0 0 0; parent root_right_hip_link0 -> root

File: urdf/humanoid.xacro (robot description, xacro)
@@ -13,6 +13,6 @@
   <link name="${parent}_${child}_link1">
     <inertial>
-      <mass value="5e-4" />
-      <inertia ixx="5e-4" ixy="0" ixz="0" iyy="5e-5" iyz="0" izz="5e-4" />
+      <mass value="1e-09" />
+      <inertia ixx="1e-09" ixy="0" ixz="0" iyy="1e-09" iyz="0" izz="1e-09" />
     </inertial>
   </link>
@@ -24,6 +24,6 @@
   <link name="${parent}_${child}_link2">
     <inertial>
-      <mass value="5e-4" />
-      <inertia ixx="5e-4" ixy="0" ixz="0" iyy="5e-5" iyz="0" izz="5e-4" />
+      <mass value="1e-09" />
+      <inertia ixx="1e-09" ixy="0" ixz="0" iyy="1e-09" iyz="0" izz="1e-09" />
     </inertial>
 	<visual>
@@ -41,6 +41,6 @@
   <link name="${parent}_${child}_link3">
     <inertial>
-      <mass value="5e-4" />
-      <inertia ixx="5e-4" ixy="0" ixz="0" iyy="5e-5" iyz="0" izz="5e-4" />
+      <mass value="1e-09" />
+      <inertia ixx="1e-09" ixy="0" ixz="0" iyy="1e-09" iyz="0" izz="1e-09" />
     </inertial>
   </link>
@@ -58,4 +58,5 @@
 	</collision>
 	<visual>
+		<xacro:insert_block name="origin"/>
 		<geometry>
 			<sphere radius="${radius/2}"/>
@@ -67,5 +68,5 @@
 		<xacro:insert_block name="origin"/>
 		<geometry>
-			<cylinder length="${length}" radius = "${radius/2}"/>
+			<cylinder length="${length*3/4}" radius = "${radius/4}"/>
 		</geometry>
 	</collision>
@@ -104,5 +105,5 @@
 			<origin rpy = "0 0 0" xyz = "0.0 0.07 0.0" />
 			<mass value = "6.000000" />
-			<inertia ixx = "0.1" ixy = "0" ixz = "0" iyy = "0.1" iyz = "0" izz = "0.1" />
+      		<inertia ixx="0.019440000000000002" ixy="0" ixz="0" iyy="0.019440000000000002" iyz="0" izz="0.019440000000000002"/>
 		</inertial>
 		<xacro:sphere_v_c radius="0.18">
@@ -119,5 +120,5 @@
 			<origin rpy = "0 0 0" xyz = "0.000000 0.120000 0.000000" />
 			<mass value = "14.000000" />
-			<inertia ixx = "0.1" ixy = "0" ixz = "0" iyy = "0.1" iyz = "0" izz = "0.1" />
+      		<inertia ixx="0.06776000000000001" ixy="0" ixz="0" iyy="0.06776000000000001" iyz="0" izz="0.06776000000000001"/>
 		</inertial>
 		<xacro:sphere_v_c radius="0.22">
@@ -132,5 +133,5 @@
 			<origin rpy = "0 0 0" xyz = "0.0 0.175 0.0" />
 			<mass value = "2.000000" />
-			<inertia ixx = "0.1" ixy = "0" ixz = "0" iyy = "0.1" iyz = "0" izz = "0.1" />
+      		<inertia ixx="0.008405" ixy="0" ixz="0" iyy="0.008405" iyz="0" izz="0.008405"/>
 		</inertial>
 		<xacro:sphere_v_c radius="0.205">
@@ -145,5 +146,5 @@
 			<origin rpy = "0 0 0" xyz = "0.000000 -0.210000 0.000000" />
 			<mass value = "4.500000" />
-			<inertia ixx = "0.1" ixy = "0" ixz = "0" iyy = "0.1" iyz = "0" izz = "0.1" />
+			<inertia ixx="0.037153124999999995" ixy="0.0" ixz="0.0" iyy="0.037153124999999995" iyz="0.0" izz="0.00680625"/>
 		</inertial>
 		<xacro:cylinder_v_c radius="0.11" length="0.3">
@@ -175,8 +176,8 @@
 			<origin rpy = "0 0 0" xyz = "0.045 -0.00225 0.000000" />
 			<mass value = "1.000000" />
-			<inertia ixx = "0.1" ixy = "0" ixz = "0" iyy = "0.1" iyz = "0" izz = "0.1" />
+			<inertia ixx="0.0009270833333333333" ixy="0.0" ixz="0.0" iyy="0.0028628333333333327" iyz="0.0" izz="0.003285749999999999"/>
 		</inertial>
 		<xacro:box_v_c x="0.177" y="0.055" z = "0.09">
-				<origin rpy = "0 0 0" xyz = "0.045 -0.00225 0.000000"  />
+			<origin rpy = "0 0 0" xyz = "0.045 -0.00225 0.000000"  />
 		</xacro:box_v_c>
 	</link>
@@ -188,5 +189,5 @@
 			<origin rpy = "0 0 0" xyz = "0.000000 -0.140000 0.000000" />
 			<mass value = "1.500000" />
-			<inertia ixx = "0.1" ixy = "0" ixz = "0" iyy = "0.1" iyz = "0" izz = "0.1" />
+			<inertia ixx="0.004809374999999999" ixy="0.0" ixz="0.0" iyy="0.004809374999999999" iyz="0.0" izz="0.0015187500000000001"/>
 		</inertial>
 		<xacro:cylinder_v_c length="0.18" radius="0.09">
@@ -201,5 +202,5 @@
 			<origin rpy = "0 0 0" xyz = "0.000000 -0.120000 0.000000" />
 			<mass value = "1.000000" />
-			<inertia ixx = "0.1" ixy = "0" ixz = "0" iyy = "0.1" iyz = "0" izz = "0.1" />
+			<inertia ixx="0.0019187499999999999" ixy="0.0" ixz="0.0" iyy="0.0019187499999999999" iyz="0.0" izz="0.0008"/>
 		</inertial>
 		<xacro:cylinder_v_c length="0.135" radius="0.08">
@@ -218,5 +219,5 @@
 			<origin rpy = "0 0 0" xyz = "0.000000 0.000000 0.000000" />
 			<mass value = "0.500000" />
-			<inertia ixx = "0.1" ixy = "0" ixz = "0" iyy = "0.1" iyz = "0" izz = "0.1" />
+			<inertia ixx="0.00032" ixy="0" ixz="0" iyy="0.00032" iyz="0" izz="0.00032"/>
 		</inertial>
 		<xacro:sphere_v_c radius="0.08">
@@ -233,5 +234,5 @@
 			<origin rpy = "0 0 0" xyz = "0.000000 -0.210000 0.000000" />
 			<mass value = "4.500000" />
-			<inertia ixx = "0.1" ixy = "0" ixz = "0" iyy = "0.1" iyz = "0" izz = "0.1" />
+			<inertia ixx="0.037153124999999995" ixy="0.0" ixz="0.0" iyy="0.037153124999999995" iyz="0.0" izz="0.00680625"/>
 		</inertial>
 		<xacro:cylinder_v_c length="0.3" radius="0.11">
@@ -244,7 +245,7 @@
 	<link name="left_knee" >
 		<inertial>
-				<origin rpy = "0 0 0" xyz = "0.000000 -0.200000 0.000000" />
-			 <mass value = "3.000000" />
-			<inertia ixx = "0.1" ixy = "0" ixz = "0" iyy = "0.1" iyz = "0" izz = "0.1" />
+			<origin rpy = "0 0 0" xyz = "0.000000 -0.200000 0.000000" />
+			<mass value = "3.000000" />
+			<inertia ixx="0.025900000000000003" ixy="0.0" ixz="0.0" iyy="0.025900000000000003" iyz="0.0" izz="0.0037500000000000007"/>
 		</inertial>
 		<xacro:cylinder_v_c length="0.31" radius="0.10000">
@@ -263,5 +264,5 @@
 			<origin rpy = "0 0 0" xyz = "0.045 -0.00225 0.0" />
 			<mass value = "1.000000" />
-			<inertia ixx = "0.1" ixy = "0" ixz = "0" iyy = "0.1" iyz = "0" izz = "0.1" />
+			<inertia ixx="0.0009270833333333333" ixy="0.0" ixz="0.0" iyy="0.0028628333333333327" iyz="0.0" izz="0.003285749999999999"/>
 		</inertial>
 		<xacro:box_v_c x="0.177" y="0.055" z = "0.09">
@@ -276,5 +277,5 @@
 			<origin rpy = "0 0 0" xyz = "0.000000 -0.140000 0.000000" />
 			<mass value = "1.500000" />
-			<inertia ixx = "0.1" ixy = "0" ixz = "0" iyy = "0.1" iyz = "0" izz = "0.1" />
+			<inertia ixx="0.004809374999999999" ixy="0.0" ixz="0.0" iyy="0.004809374999999999" iyz="0.0" izz="0.0015187500000000001"/>
 		</inertial>
 		<xacro:cylinder_v_c length="0.18" radius="0.09">
@@ -289,5 +290,5 @@
 			<origin rpy = "0 0 0" xyz = "0.000000 -0.12 0.000000" />
 			<mass value = "1.000000" />
-			<inertia ixx = "0.1" ixy = "0" ixz = "0" iyy = "0.1" iyz = "0" izz = "0.1" />
+			<inertia ixx="0.0019187499999999999" ixy="0.0" ixz="0.0" iyy="0.0019187499999999999" iyz="0.0" izz="0.0008"/>
 		</inertial>
 		<xacro:cylinder_v_c length="0.135" radius="0.08">
@@ -306,5 +307,5 @@
 			<origin rpy = "0 0 0" xyz = "0.000000 0.000000 0.000000" />
 			<mass value = "0.500000" />
-			<inertia ixx = "0.1" ixy = "0" ixz = "0" iyy = "0.1" iyz = "0" izz = "0.1" />
+			<inertia ixx="0.00032" ixy="0" ixz="0" iyy="0.00032" iyz="0" izz="0.00032"/>
 		</inertial>
 		<xacro:sphere_v_c radius="0.08">

Commit message: Remove useless virtual link and fixed joint in shperical joints

File: urdf/humanoid.urdf (robot description, URDF)
Before this commit: robot dumpUrdf, 41 links, 40 joints
Links:
- removed link chest_left_shoulder_link3
- removed link chest_neck_link3
- removed link chest_right_shoulder_link3
- removed link left_knee_left_ankle_link3
- removed link right_knee_right_ankle_link3
- removed link root_chest_link3
- removed link root_left_hip_link3
- removed link root_right_hip_link3
- link chest_left_shoulder_link1: mass 1e-09 -> 1e-02
- link chest_left_shoulder_link2: mass 1e-09 -> 1e-02
- link chest_neck_link1: mass 1e-09 -> 1e-02
- link chest_neck_link2: mass 1e-09 -> 1e-02
- link chest_right_shoulder_link1: mass 1e-09 -> 1e-02
- link chest_right_shoulder_link2: mass 1e-09 -> 1e-02
- link left_knee_left_ankle_link1: mass 1e-09 -> 1e-02
- link left_knee_left_ankle_link2: mass 1e-09 -> 1e-02
- link right_knee_right_ankle_link1: mass 1e-09 -> 1e-02
- link right_knee_right_ankle_link2: mass 1e-09 -> 1e-02
- link root_chest_link1: mass 1e-09 -> 1e-02
- link root_chest_link2: mass 1e-09 -> 1e-02
- link root_left_hip_link1: mass 1e-09 -> 1e-02
- link root_left_hip_link2: mass 1e-09 -> 1e-02
- link root_right_hip_link1: mass 1e-09 -> 1e-02
- link root_right_hip_link2: mass 1e-09 -> 1e-02
Joints:
- removed joint chest_left_shoulder_joint4
- removed joint chest_neck_joint4
- removed joint chest_right_shoulder_joint4
- removed joint left_knee_left_ankle_joint4
- removed joint right_knee_right_ankle_joint4
- removed joint root_chest_joint4
- removed joint root_left_hip_joint4
- removed joint root_right_hip_joint4
- joint chest_left_shoulder_joint3: child chest_left_shoulder_link3 -> left_shoulder
- joint chest_neck_joint3: child chest_neck_link3 -> neck
- joint chest_right_shoulder_joint3: child chest_right_shoulder_link3 -> right_shoulder
- joint left_knee_left_ankle_joint3: child left_knee_left_ankle_link3 -> left_ankle
- joint right_knee_right_ankle_joint3: child right_knee_right_ankle_link3 -> right_ankle
- joint root_chest_joint3: child root_chest_link3 -> chest
- joint root_left_hip_joint3: child root_left_hip_link3 -> left_hip
- joint root_right_hip_joint3: child root_right_hip_link3 -> right_hip

File: urdf/humanoid.xacro (robot description, xacro)
@@ -36,16 +36,6 @@
   <joint name="${parent}_${child}_joint3" type="continuous">
     <parent link="${parent}_${child}_link2"/>
-    <child link="${parent}_${child}_link3"/>
+    <child link="${child}"/>
     <axis xyz="0 0 1" />
-  </joint>
-  <link name="${parent}_${child}_link3">
-    <inertial>
-      <mass value="1e-02" />
-      <inertia ixx="1e-02" ixy="0" ixz="0" iyy="1e-02" iyz="0" izz="1e-02" />
-    </inertial>
-  </link>
-  <joint name="${parent}_${child}_joint4" type="fixed">
-    <parent link="${parent}_${child}_link3"/>
-    <child link="${child}"/>
   </joint>
 </xacro:macro>

Commit message: replace three revolute joints with one spherical one for RaiSim physics engine

File: urdf/humanoid.urdf (robot description, URDF)
Before this commit: robot dumpUrdf, 33 links, 32 joints
Links:
- removed link chest_left_shoulder_link1
- removed link chest_left_shoulder_link2
- removed link chest_neck_link1
- removed link chest_neck_link2
- removed link chest_right_shoulder_link1
- removed link chest_right_shoulder_link2
- removed link left_knee_left_ankle_link1
- removed link left_knee_left_ankle_link2
- removed link right_knee_right_ankle_link1
- removed link right_knee_right_ankle_link2
- removed link root_chest_link1
- removed link root_chest_link2
- removed link root_left_hip_link1
- removed link root_left_hip_link2
- removed link root_right_hip_link1
- removed link root_right_hip_link2
Joints:
- removed joint chest_left_shoulder_joint1
- removed joint chest_left_shoulder_joint2
- removed joint chest_left_shoulder_joint3
- removed joint chest_neck_joint1
- removed joint chest_neck_joint2
- removed joint chest_neck_joint3
- removed joint chest_right_shoulder_joint1
- removed joint chest_right_shoulder_joint2
- removed joint chest_right_shoulder_joint3
- removed joint left_knee_left_ankle_joint1
- removed joint left_knee_left_ankle_joint2
- removed joint left_knee_left_ankle_joint3
- removed joint right_knee_right_ankle_joint1
- removed joint right_knee_right_ankle_joint2
- removed joint right_knee_right_ankle_joint3
- removed joint root_chest_joint1
- removed joint root_chest_joint2
- removed joint root_chest_joint3
- removed joint root_left_hip_joint1
- removed joint root_left_hip_joint2
- removed joint root_left_hip_joint3
- removed joint root_right_hip_joint1
- removed joint root_right_hip_joint2
- removed joint root_right_hip_joint3
- added joint chest_left_shoulder: type spherical, parent chest, child left_shoulder, origin xyz=-0.02405 0.24350 -0.18311 rpy=0 0 0, axis 0 1 0
- added joint chest_neck: type spherical, parent chest, child neck, origin xyz=0.000000 0.223894 0.000000 rpy=0 0 0, axis 0 1 0
- added joint chest_right_shoulder: type spherical, parent chest, child right_shoulder, origin xyz=-0.02406 0.24350 0.18311 rpy=0 0 0, axis 0 1 0
- added joint left_knee_left_ankle: type spherical, parent left_knee, child left_ankle, origin xyz=0.000000 -0.40987 0.000000 rpy=0 0 0, axis 0 1 0
- added joint right_knee_right_ankle: type spherical, parent right_knee, child right_ankle, origin xyz=0.000000 -0.409870 0.000000 rpy=0 0 0, axis 0 1 0
- added joint root_chest: type spherical, parent root, child chest, origin xyz=0.000000 0.236151 0.000000 rpy=0 0 0, axis 0 1 0
- added joint root_left_hip: type spherical, parent root, child left_hip, origin xyz=0.000000 0.000000 -0.084887 rpy=0 0 0, axis 0 1 0
- added joint root_right_hip: type spherical, parent root, child right_hip, origin xyz=0.000000 0.000000 0.084887 rpy=0 0 0, axis 0 1 0

File: urdf/humanoid.xacro (robot description, xacro)
@@ -5,37 +5,9 @@
 </material>
 <xacro:macro name="ball_joint" params="parent child *origin">
-  <joint name="${parent}_${child}_joint1" type="continuous">
+  <joint name="${parent}_${child}" type="spherical">
+	<parent link="${parent}"/>
+	<child link="${child}"/>
 	<xacro:insert_block name="origin"/>
-    <parent link="${parent}"/>
-    <child link="${parent}_${child}_link1"/>
-    <axis xyz="1 0 0" />
-  </joint>
-  <link name="${parent}_${child}_link1">
-    <inertial>
-      <mass value="1e-02" />
-      <inertia ixx="1e-02" ixy="0" ixz="0" iyy="1e-02" iyz="0" izz="1e-02" />
-    </inertial>
-  </link>
-  <joint name="${parent}_${child}_joint2" type="continuous">
-    <parent link="${parent}_${child}_link1"/>
-    <child link="${parent}_${child}_link2"/>
-    <axis xyz="0 1 0" />
-  </joint>
-  <link name="${parent}_${child}_link2">
-    <inertial>
-      <mass value="1e-02" />
-      <inertia ixx="1e-02" ixy="0" ixz="0" iyy="1e-02" iyz="0" izz="1e-02" />
-    </inertial>
-	<visual>
-		<geometry>
-			<sphere radius="0.05"  />
-		</geometry>
-		<material name="orange"/>
-	</visual>
-  </link>
-  <joint name="${parent}_${child}_joint3" type="continuous">
-    <parent link="${parent}_${child}_link2"/>
-    <child link="${child}"/>
-    <axis xyz="0 0 1" />
+	<axis xyz="0 1 0"/>
   </joint>
 </xacro:macro>
