Commit message: Add limits to effort and range

File: urdf/humanoid.urdf (robot description, URDF)
Before this commit: robot dumpUrdf, 33 links, 32 joints
Joints:
- joint chest_left_shoulder_joint1: limit (none) -> lower=3.14 upper=3.14 effort=100
- joint chest_left_shoulder_joint2: limit (none) -> lower=3.14 upper=3.14 effort=100
- joint chest_left_shoulder_joint3: limit (none) -> lower=3.14 upper=3.14 effort=100
- joint chest_neck_joint1: limit (none) -> lower=1 upper=1 effort=50
- joint chest_neck_joint2: limit (none) -> lower=1 upper=1 effort=50
- joint chest_neck_joint3: limit (none) -> lower=1 upper=1 effort=50
- joint chest_right_shoulder_joint1: limit (none) -> lower=3.14 upper=3.14 effort=100
- joint chest_right_shoulder_joint2: limit (none) -> lower=3.14 upper=3.14 effort=100
- joint chest_right_shoulder_joint3: limit (none) -> lower=3.14 upper=3.14 effort=100
- joint left_elbow: limit lower=0 upper=3.14 effort=1000.0 velocity=0.5 -> lower=0 upper=3.14 effort=60.0 velocity=0.5
- joint left_knee: limit lower=-3.14 upper=0. effort=1000.0 velocity=0.5 -> lower=-3.14 upper=0. effort=150.0 velocity=0.5
- joint left_knee_left_ankle_joint1: limit (none) -> lower=1.2 upper=1.2 effort=90
- joint left_knee_left_ankle_joint2: limit (none) -> lower=1.2 upper=1.2 effort=90
- joint left_knee_left_ankle_joint3: limit (none) -> lower=1.2 upper=1.2 effort=90
- joint right_elbow: limit lower=0 upper=3.14 effort=1000.0 velocity=0.5 -> lower=0 upper=3.14 effort=60.0 velocity=0.5
- joint right_knee: limit lower=-3.14 upper=0. effort=1000.0 velocity=0.5 -> lower=-3.14 upper=0. effort=150.0 velocity=0.5
- joint right_knee_right_ankle_joint1: limit (none) -> lower=1.2 upper=1.2 effort=90
- joint right_knee_right_ankle_joint2: limit (none) -> lower=1.2 upper=1.2 effort=90
- joint right_knee_right_ankle_joint3: limit (none) -> lower=1.2 upper=1.2 effort=90
- joint root_chest_joint1: limit (none) -> lower=1.2 upper=1.2 effort=200
- joint root_chest_joint2: limit (none) -> lower=1.2 upper=1.2 effort=200
- joint root_chest_joint3: limit (none) -> lower=1.2 upper=1.2 effort=200
- joint root_left_hip_joint1: limit (none) -> lower=1.5 upper=1.5 effort=200
- joint root_left_hip_joint2: limit (none) -> lower=1.5 upper=1.5 effort=200
- joint root_left_hip_joint3: limit (none) -> lower=1.5 upper=1.5 effort=200
- joint root_right_hip_joint1: limit (none) -> lower=1.5 upper=1.5 effort=200
- joint root_right_hip_joint2: limit (none) -> lower=1.5 upper=1.5 effort=200
- joint root_right_hip_joint3: limit (none) -> lower=1.5 upper=1.5 effort=200

File: urdf/humanoid.xacro (robot description, xacro)
@@ -4,5 +4,5 @@
   <color rgba="${255/255} ${108/255} ${10/255} 1.0"/>
 </material>
-<xacro:macro name="ball_joint" params="parent child *origin">
+<xacro:macro name="ball_joint" params="parent child limit effort_limit *origin">
   <link name="${parent}_${child}_link1">
     <inertial>
@@ -16,4 +16,5 @@
     <child link="${parent}_${child}_link1"/>
     <axis xyz="1 0 0" />
+	<limit effort="${effort_limit}" lower="${limit}" upper="${limit}"/>
   </joint>
   <link name="${parent}_${child}_link2">
@@ -33,4 +34,5 @@
     <child link="${parent}_${child}_link2"/>
     <axis xyz="0 1 0" />
+	<limit effort="${effort_limit}" lower="${limit}" upper="${limit}"/>
   </joint>
   <joint name="${parent}_${child}_joint3" type="continuous">
@@ -38,4 +40,5 @@
     <child link="${child}"/>
     <axis xyz="0 0 1" />
+	<limit effort="${effort_limit}" lower="${limit}" upper="${limit}"/>
   </joint>
 </xacro:macro>
@@ -116,5 +119,5 @@
 		</xacro:sphere_v_c>
 	</link>
-	<xacro:ball_joint parent="root" child="chest">
+	<xacro:ball_joint parent="root" child="chest" limit="1.2" effort_limit="200">
 		<origin rpy = "0 0 0" xyz = "0.000000 0.236151 0.000000" />
 	</xacro:ball_joint>
@@ -129,5 +132,5 @@
 		</xacro:sphere_v_c>
 	</link>
-	<xacro:ball_joint parent="chest" child="neck" >
+	<xacro:ball_joint parent="chest" child="neck" limit="1" effort_limit="50" >
 		<origin rpy = "0 0 0" xyz = "0.000000 0.223894 0.000000" />
 	</xacro:ball_joint>
@@ -142,5 +145,5 @@
 		</xacro:cylinder_v_c>
 	</link>
-	<xacro:ball_joint parent="root" child="right_hip">
+	<xacro:ball_joint parent="root" child="right_hip" limit="1.5" effort_limit="200">
 		<origin rpy = "0 0 0" xyz = "0.000000 0.000000 0.084887" />
 	</xacro:ball_joint>
@@ -158,5 +161,5 @@
 		<parent link="right_hip" />
 		<child link="right_knee" />
-		<limit effort="1000.0" lower="-3.14" upper="0." velocity="0.5"/>
+		<limit effort="150.0" lower="-3.14" upper="0." velocity="0.5"/>
 		<origin rpy = "0 0 0" xyz = "0.000000 -0.421546 0.000000" />
 		<axis xyz = "0.000000 0.000000 1.000000" />
@@ -172,5 +175,5 @@
 		</xacro:box_v_c>
 	</link>
-	<xacro:ball_joint parent="right_knee" child="right_ankle">
+	<xacro:ball_joint parent="right_knee" child="right_ankle" limit="1.2" effort_limit="90">
 		<origin rpy = "0 0 0" xyz = "0.000000 -0.409870 0.000000" />
 	</xacro:ball_joint>
@@ -185,5 +188,5 @@
 		</xacro:cylinder_v_c>
 	</link>
-	<xacro:ball_joint parent="chest" child="right_shoulder">
+	<xacro:ball_joint parent="chest" child="right_shoulder" limit="3.14" effort_limit="100">
 		<origin rpy = "0 0 0" xyz = "-0.02406 0.24350 0.18311" />
 	</xacro:ball_joint>
@@ -201,5 +204,5 @@
 		<parent link="right_shoulder" />
 		<child link="right_elbow" />
-		<limit effort="1000.0" lower="0" upper="3.14" velocity="0.5"/>
+		<limit effort="60.0" lower="0" upper="3.14" velocity="0.5"/>
 		<origin rpy = "0 0 0" xyz = "0.000000 -0.274788 0.000000" />
 		<axis xyz = "0.000000 0.000000 1.000000" />
@@ -230,5 +233,5 @@
 		</xacro:cylinder_v_c>
 	</link>
-	<xacro:ball_joint parent="root" child="left_hip">
+	<xacro:ball_joint parent="root" child="left_hip" limit="1.5" effort_limit="200">
 		<origin rpy = "0 0 0" xyz = "0.000000 0.000000 -0.084887" />
 	</xacro:ball_joint>
@@ -246,5 +249,5 @@
 		<parent link="left_hip" />
 		<child link="left_knee" />
-		<limit effort="1000.0" lower="-3.14" upper="0." velocity="0.5"/>
+		<limit effort="150.0" lower="-3.14" upper="0." velocity="0.5"/>
 		<origin rpy = "0 0 0" xyz = "0.000000 -0.421546 0.000000" />
 		<axis xyz = "0.000000 0.000000 1.000000" />
@@ -260,5 +263,5 @@
 		</xacro:box_v_c>
 	</link>
-	<xacro:ball_joint parent="left_knee" child="left_ankle">
+	<xacro:ball_joint parent="left_knee" child="left_ankle" limit="1.2" effort_limit="90">
 		<origin rpy = "0 0 0" xyz = "0.000000 -0.40987 0.000000" />
 	</xacro:ball_joint>
@@ -273,5 +276,5 @@
 		</xacro:cylinder_v_c>
 	</link>
-	<xacro:ball_joint parent="chest" child="left_shoulder">
+	<xacro:ball_joint parent="chest" child="left_shoulder" limit="3.14" effort_limit="100">
 		<origin rpy = "0 0 0" xyz = "-0.02405 0.24350 -0.18311" />
 	</xacro:ball_joint>
@@ -289,5 +292,5 @@
 		<parent link="left_shoulder" />
 		<child link="left_elbow" />
-		<limit effort="1000.0" lower="0" upper="3.14" velocity="0.5"/>
+		<limit effort="60.0" lower="0" upper="3.14" velocity="0.5"/>
 		<origin rpy = "0 0 0" xyz = "0.000000 -0.274788 0.000000" />
 		<axis xyz = "0.000000 0.000000 1.000000" />

Commit message: Fix lower limit

File: urdf/humanoid.urdf (robot description, URDF)
Before this commit: robot dumpUrdf, 33 links, 32 joints
Joints:
- joint chest_left_shoulder_joint1: limit lower=3.14 upper=3.14 effort=100 -> lower=-3.14 upper=3.14 effort=100
- joint chest_left_shoulder_joint2: limit lower=3.14 upper=3.14 effort=100 -> lower=-3.14 upper=3.14 effort=100
- joint chest_left_shoulder_joint3: limit lower=3.14 upper=3.14 effort=100 -> lower=-3.14 upper=3.14 effort=100
- joint chest_neck_joint1: limit lower=1 upper=1 effort=50 -> lower=-1 upper=1 effort=50
- joint chest_neck_joint2: limit lower=1 upper=1 effort=50 -> lower=-1 upper=1 effort=50
- joint chest_neck_joint3: limit lower=1 upper=1 effort=50 -> lower=-1 upper=1 effort=50
- joint chest_right_shoulder_joint1: limit lower=3.14 upper=3.14 effort=100 -> lower=-3.14 upper=3.14 effort=100
- joint chest_right_shoulder_joint2: limit lower=3.14 upper=3.14 effort=100 -> lower=-3.14 upper=3.14 effort=100
- joint chest_right_shoulder_joint3: limit lower=3.14 upper=3.14 effort=100 -> lower=-3.14 upper=3.14 effort=100
- joint left_knee_left_ankle_joint1: limit lower=1.2 upper=1.2 effort=90 -> lower=-1.2 upper=1.2 effort=90
- joint left_knee_left_ankle_joint2: limit lower=1.2 upper=1.2 effort=90 -> lower=-1.2 upper=1.2 effort=90
- joint left_knee_left_ankle_joint3: limit lower=1.2 upper=1.2 effort=90 -> lower=-1.2 upper=1.2 effort=90
- joint right_knee_right_ankle_joint1: limit lower=1.2 upper=1.2 effort=90 -> lower=-1.2 upper=1.2 effort=90
- joint right_knee_right_ankle_joint2: limit lower=1.2 upper=1.2 effort=90 -> lower=-1.2 upper=1.2 effort=90
- joint right_knee_right_ankle_joint3: limit lower=1.2 upper=1.2 effort=90 -> lower=-1.2 upper=1.2 effort=90
- joint root_chest_joint1: limit lower=1.2 upper=1.2 effort=200 -> lower=-1.2 upper=1.2 effort=200
- joint root_chest_joint2: limit lower=1.2 upper=1.2 effort=200 -> lower=-1.2 upper=1.2 effort=200
- joint root_chest_joint3: limit lower=1.2 upper=1.2 effort=200 -> lower=-1.2 upper=1.2 effort=200
- joint root_left_hip_joint1: limit lower=1.5 upper=1.5 effort=200 -> lower=-1.5 upper=1.5 effort=200
- joint root_left_hip_joint2: limit lower=1.5 upper=1.5 effort=200 -> lower=-1.5 upper=1.5 effort=200
- joint root_left_hip_joint3: limit lower=1.5 upper=1.5 effort=200 -> lower=-1.5 upper=1.5 effort=200
- joint root_right_hip_joint1: limit lower=1.5 upper=1.5 effort=200 -> lower=-1.5 upper=1.5 effort=200
- joint root_right_hip_joint2: limit lower=1.5 upper=1.5 effort=200 -> lower=-1.5 upper=1.5 effort=200
- joint root_right_hip_joint3: limit lower=1.5 upper=1.5 effort=200 -> lower=-1.5 upper=1.5 effort=200

File: urdf/humanoid.xacro (robot description, xacro)
@@ -16,5 +16,5 @@
     <child link="${parent}_${child}_link1"/>
     <axis xyz="1 0 0" />
-	<limit effort="${effort_limit}" lower="${limit}" upper="${limit}"/>
+	<limit effort="${effort_limit}" lower="${-limit}" upper="${limit}"/>
   </joint>
   <link name="${parent}_${child}_link2">
@@ -34,5 +34,5 @@
     <child link="${parent}_${child}_link2"/>
     <axis xyz="0 1 0" />
-	<limit effort="${effort_limit}" lower="${limit}" upper="${limit}"/>
+	<limit effort="${effort_limit}" lower="${-limit}" upper="${limit}"/>
   </joint>
   <joint name="${parent}_${child}_joint3" type="continuous">
@@ -40,5 +40,5 @@
     <child link="${child}"/>
     <axis xyz="0 0 1" />
-	<limit effort="${effort_limit}" lower="${limit}" upper="${limit}"/>
+	<limit effort="${effort_limit}" lower="${-limit}" upper="${limit}"/>
   </joint>
 </xacro:macro>

Commit message: Fix lower limit

File: urdf/humanoid.urdf (robot description, URDF)
Before this commit: robot dumpUrdf, 33 links, 32 joints
Joints:
- joint chest_left_shoulder_joint1: type continuous -> revolute
- joint chest_left_shoulder_joint2: type continuous -> revolute
- joint chest_left_shoulder_joint3: type continuous -> revolute
- joint chest_neck_joint1: type continuous -> revolute
- joint chest_neck_joint2: type continuous -> revolute
- joint chest_neck_joint3: type continuous -> revolute
- joint chest_right_shoulder_joint1: type continuous -> revolute
- joint chest_right_shoulder_joint2: type continuous -> revolute
- joint chest_right_shoulder_joint3: type continuous -> revolute
- joint left_knee_left_ankle_joint1: type continuous -> revolute
- joint left_knee_left_ankle_joint2: type continuous -> revolute
- joint left_knee_left_ankle_joint3: type continuous -> revolute
- joint right_knee_right_ankle_joint1: type continuous -> revolute
- joint right_knee_right_ankle_joint2: type continuous -> revolute
- joint right_knee_right_ankle_joint3: type continuous -> revolute
- joint root_chest_joint1: type continuous -> revolute
- joint root_chest_joint2: type continuous -> revolute
- joint root_chest_joint3: type continuous -> revolute
- joint root_left_hip_joint1: type continuous -> revolute
- joint root_left_hip_joint2: type continuous -> revolute
- joint root_left_hip_joint3: type continuous -> revolute
- joint root_right_hip_joint1: type continuous -> revolute
- joint root_right_hip_joint2: type continuous -> revolute
- joint root_right_hip_joint3: type continuous -> revolute

File: urdf/humanoid.xacro (robot description, xacro)
@@ -11,5 +11,5 @@
     </inertial>
   </link>
-  <joint name="${parent}_${child}_joint1" type="continuous">
+  <joint name="${parent}_${child}_joint1" type="revolute">
 	<xacro:insert_block name="origin"/>
     <parent link="${parent}"/>
@@ -30,5 +30,5 @@
 	</visual>
   </link>
-  <joint name="${parent}_${child}_joint2" type="continuous">
+  <joint name="${parent}_${child}_joint2" type="revolute">
     <parent link="${parent}_${child}_link1"/>
     <child link="${parent}_${child}_link2"/>
@@ -36,5 +36,5 @@
 	<limit effort="${effort_limit}" lower="${-limit}" upper="${limit}"/>
   </joint>
-  <joint name="${parent}_${child}_joint3" type="continuous">
+  <joint name="${parent}_${child}_joint3" type="revolute">
     <parent link="${parent}_${child}_link2"/>
     <child link="${child}"/>

Commit message: Add a velocity limit

File: urdf/humanoid.urdf (robot description, URDF)
Before this commit: robot dumpUrdf, 33 links, 32 joints
Joints:
- joint chest_left_shoulder_joint1: limit lower=-3.14 upper=3.14 effort=100 -> lower=-3.14 upper=3.14 effort=100 velocity=3
- joint chest_left_shoulder_joint2: limit lower=-3.14 upper=3.14 effort=100 -> lower=-3.14 upper=3.14 effort=100 velocity=3
- joint chest_left_shoulder_joint3: limit lower=-3.14 upper=3.14 effort=100 -> lower=-3.14 upper=3.14 effort=100 velocity=3
- joint chest_neck_joint1: limit lower=-1 upper=1 effort=50 -> lower=-1 upper=1 effort=50 velocity=3
- joint chest_neck_joint2: limit lower=-1 upper=1 effort=50 -> lower=-1 upper=1 effort=50 velocity=3
- joint chest_neck_joint3: limit lower=-1 upper=1 effort=50 -> lower=-1 upper=1 effort=50 velocity=3
- joint chest_right_shoulder_joint1: limit lower=-3.14 upper=3.14 effort=100 -> lower=-3.14 upper=3.14 effort=100 velocity=3
- joint chest_right_shoulder_joint2: limit lower=-3.14 upper=3.14 effort=100 -> lower=-3.14 upper=3.14 effort=100 velocity=3
- joint chest_right_shoulder_joint3: limit lower=-3.14 upper=3.14 effort=100 -> lower=-3.14 upper=3.14 effort=100 velocity=3
- joint left_knee_left_ankle_joint1: limit lower=-1.2 upper=1.2 effort=90 -> lower=-1.2 upper=1.2 effort=90 velocity=3
- joint left_knee_left_ankle_joint2: limit lower=-1.2 upper=1.2 effort=90 -> lower=-1.2 upper=1.2 effort=90 velocity=3
- joint left_knee_left_ankle_joint3: limit lower=-1.2 upper=1.2 effort=90 -> lower=-1.2 upper=1.2 effort=90 velocity=3
- joint right_knee_right_ankle_joint1: limit lower=-1.2 upper=1.2 effort=90 -> lower=-1.2 upper=1.2 effort=90 velocity=3
- joint right_knee_right_ankle_joint2: limit lower=-1.2 upper=1.2 effort=90 -> lower=-1.2 upper=1.2 effort=90 velocity=3
- joint right_knee_right_ankle_joint3: limit lower=-1.2 upper=1.2 effort=90 -> lower=-1.2 upper=1.2 effort=90 velocity=3
- joint root_chest_joint1: limit lower=-1.2 upper=1.2 effort=200 -> lower=-1.2 upper=1.2 effort=200 velocity=3
- joint root_chest_joint2: limit lower=-1.2 upper=1.2 effort=200 -> lower=-1.2 upper=1.2 effort=200 velocity=3
- joint root_chest_joint3: limit lower=-1.2 upper=1.2 effort=200 -> lower=-1.2 upper=1.2 effort=200 velocity=3
- joint root_left_hip_joint1: limit lower=-1.5 upper=1.5 effort=200 -> lower=-1.5 upper=1.5 effort=200 velocity=3
- joint root_left_hip_joint2: limit lower=-1.5 upper=1.5 effort=200 -> lower=-1.5 upper=1.5 effort=200 velocity=3
- joint root_left_hip_joint3: limit lower=-1.5 upper=1.5 effort=200 -> lower=-1.5 upper=1.5 effort=200 velocity=3
- joint root_right_hip_joint1: limit lower=-1.5 upper=1.5 effort=200 -> lower=-1.5 upper=1.5 effort=200 velocity=3
- joint root_right_hip_joint2: limit lower=-1.5 upper=1.5 effort=200 -> lower=-1.5 upper=1.5 effort=200 velocity=3
- joint root_right_hip_joint3: limit lower=-1.5 upper=1.5 effort=200 -> lower=-1.5 upper=1.5 effort=200 velocity=3

File: urdf/humanoid.xacro (robot description, xacro)
@@ -16,5 +16,5 @@
     <child link="${parent}_${child}_link1"/>
     <axis xyz="1 0 0" />
-	<limit effort="${effort_limit}" lower="${-limit}" upper="${limit}"/>
+	<limit effort="${effort_limit}" lower="${-limit}" upper="${limit}" velocity="3"/>
   </joint>
   <link name="${parent}_${child}_link2">
@@ -34,5 +34,5 @@
     <child link="${parent}_${child}_link2"/>
     <axis xyz="0 1 0" />
-	<limit effort="${effort_limit}" lower="${-limit}" upper="${limit}"/>
+	<limit effort="${effort_limit}" lower="${-limit}" upper="${limit}" velocity="3"/>
   </joint>
   <joint name="${parent}_${child}_joint3" type="revolute">
@@ -40,5 +40,5 @@
     <child link="${child}"/>
     <axis xyz="0 0 1" />
-	<limit effort="${effort_limit}" lower="${-limit}" upper="${limit}"/>
+	<limit effort="${effort_limit}" lower="${-limit}" upper="${limit}" velocity="3"/>
   </joint>
 </xacro:macro>
